File: protoboard.sch (KiCad schematic (older format))
At the start: 38 parts, among them J1 ⊕, J101 a, J102 b, J103 c, J104 d, J105 e, J106 f, J107 g, J108 h, J109 i, J110 j, J111 k, J112 l, J113 m, J114 n, J115 o, J116 p, J117 q, J118 r, J119 s, J120 t, J121 u, J122 v, J123 w, J124 x, J2 ⊕, J3 ⊕, J4 ⊕, J5 ⊖, J6 ⊖, J7 ⊖, J8 ⊖

Commit message: ready to release
Connections:
- net VCC1: now reaches J1.1 (Pin_1), J1.10 (Pin_10), J1.11 (Pin_11), J1.12 (Pin_12), J1.13 (Pin_13), J1.14 (Pin_14), J1.15 (Pin_15), J1.16 (Pin_16), J1.17 (Pin_17), J1.18 (Pin_18), J1.19 (Pin_19), J1.2 (Pin_2), J1.20 (Pin_20), J1.21 (Pin_21), J1.22 (Pin_22), J1.23 (Pin_23), J1.24 (Pin_24), J1.25 (Pin_25), J1.26 (Pin_26), J1.27 (Pin_27), J1.28 (Pin_28), J1.29 (Pin_29), J1.3 (Pin_3), J1.30 (Pin_30), J1.31 (Pin_31), J1.32 (Pin_32), J1.33 (Pin_33), J1.34 (Pin_34), J1.4 (Pin_4), J1.5 (Pin_5), J1.6 (Pin_6), J1.7 (Pin_7), J1.8 (Pin_8), J1.9 (Pin_9), J2.1 (Pin_1), J2.2 (Pin_2), J2.3 (Pin_3), J2.4 (Pin_4), J2.5 (Pin_5), J2.6 (Pin_6), JP101.1 (A)
- net VCC2: now reaches J3.1 (Pin_1), J3.10 (Pin_10), J3.11 (Pin_11), J3.12 (Pin_12), J3.13 (Pin_13), J3.14 (Pin_14), J3.15 (Pin_15), J3.16 (Pin_16), J3.17 (Pin_17), J3.18 (Pin_18), J3.19 (Pin_19), J3.2 (Pin_2), J3.20 (Pin_20), J3.21 (Pin_21), J3.22 (Pin_22), J3.23 (Pin_23), J3.24 (Pin_24), J3.25 (Pin_25), J3.26 (Pin_26), J3.27 (Pin_27), J3.28 (Pin_28), J3.29 (Pin_29), J3.3 (Pin_3), J3.30 (Pin_30), J3.31 (Pin_31), J3.32 (Pin_32), J3.33 (Pin_33), J3.34 (Pin_34), J3.4 (Pin_4), J3.5 (Pin_5), J3.6 (Pin_6), J3.7 (Pin_7), J3.8 (Pin_8), J3.9 (Pin_9), J4.1 (Pin_1), J4.2 (Pin_2), J4.3 (Pin_3), J4.4 (Pin_4), J4.5 (Pin_5), J4.6 (Pin_6), JP101.2 (B)
- net GND1: now reaches J5.1 (Pin_1), J5.10 (Pin_10), J5.11 (Pin_11), J5.12 (Pin_12), J5.13 (Pin_13), J5.14 (Pin_14), J5.15 (Pin_15), J5.16 (Pin_16), J5.17 (Pin_17), J5.18 (Pin_18), J5.19 (Pin_19), J5.2 (Pin_2), J5.20 (Pin_20), J5.21 (Pin_21), J5.22 (Pin_22), J5.23 (Pin_23), J5.24 (Pin_24), J5.25 (Pin_25), J5.26 (Pin_26), J5.27 (Pin_27), J5.28 (Pin_28), J5.29 (Pin_29), J5.3 (Pin_3), J5.30 (Pin_30), J5.31 (Pin_31), J5.32 (Pin_32), J5.33 (Pin_33), J5.34 (Pin_34), J5.4 (Pin_4), J5.5 (Pin_5), J5.6 (Pin_6), J5.7 (Pin_7), J5.8 (Pin_8), J5.9 (Pin_9), J6.1 (Pin_1), J6.2 (Pin_2), J6.3 (Pin_3), J6.4 (Pin_4), J6.5 (Pin_5), J6.6 (Pin_6), JP102.1 (A)
- net GND2: now reaches J7.1 (Pin_1), J7.10 (Pin_10), J7.11 (Pin_11), J7.12 (Pin_12), J7.13 (Pin_13), J7.14 (Pin_14), J7.15 (Pin_15), J7.16 (Pin_16), J7.17 (Pin_17), J7.18 (Pin_18), J7.19 (Pin_19), J7.2 (Pin_2), J7.20 (Pin_20), J7.21 (Pin_21), J7.22 (Pin_22), J7.23 (Pin_23), J7.24 (Pin_24), J7.25 (Pin_25), J7.26 (Pin_26), J7.27 (Pin_27), J7.28 (Pin_28), J7.29 (Pin_29), J7.3 (Pin_3), J7.30 (Pin_30), J7.31 (Pin_31), J7.32 (Pin_32), J7.33 (Pin_33), J7.34 (Pin_34), J7.4 (Pin_4), J7.5 (Pin_5), J7.6 (Pin_6), J7.7 (Pin_7), J7.8 (Pin_8), J7.9 (Pin_9), J8.1 (Pin_1), J8.2 (Pin_2), J8.3 (Pin_3), J8.4 (Pin_4), J8.5 (Pin_5), J8.6 (Pin_6), JP102.2 (B)
Changed lines of the file:
@@
 Sheet 1 1
 Title "Protoboard"
-Date "2022-09-16"
+Date "2022-10-07"
 Rev "v1.0.0"
 Comp "Sporniket"
@@
 Wire Wire Line
 	12650 5800 12650 6200
+Text Label 9150 1600 2    50   ~ 0
+VCC1
+Text Label 10150 1600 2    50   ~ 0
+VCC2
+Text Label 11650 1600 2    50   ~ 0
+GND1
+Text Label 12650 1600 2    50   ~ 0
+GND2
 Wire Bus Line
 	3750 5900 3750 9400
