File: protoboard.kicad_sch (KiCad schematic)
At the start: 38 parts, among them J1 ⊕, J101 a, J102 b, J103 c, J104 d, J105 e, J106 f, J107 g, J108 h, J109 i, J110 j, J111 k, J112 l, J113 m, J114 n, J115 o, J116 p, J117 q, J118 r, J119 s, J120 t, J121 u, J122 v, J123 w, J124 x, J2 ⊕, J3 ⊕, J4 ⊕, J5 ⊖, J6 ⊖, J7 ⊖, J8 ⊖

Commit message: wip -- reworking prototyping area
Parts:
- added J201: g1, protoboard:rows_of_pins_1x34, symbol Connector_Generic:Conn_01x34
- added J202: g2, protoboard:rows_of_pins_1x34, symbol Connector_Generic:Conn_01x34
- added J203: g3, protoboard:rows_of_pins_1x34, symbol Connector_Generic:Conn_01x34
- added J204: g4, protoboard:rows_of_pins_1x34, symbol Connector_Generic:Conn_01x34
- added J205: a1, symbol Connector_Generic:Conn_01x21
- added J206: b1, symbol Connector_Generic:Conn_01x21
- added J207: c1, symbol Connector_Generic:Conn_01x21
- added J208: d1, symbol Connector_Generic:Conn_01x21
- added J209: e1, symbol Connector_Generic:Conn_01x21
- added J210: f1, symbol Connector_Generic:Conn_01x21
- added J211: g1, symbol Connector_Generic:Conn_01x21
- added J212: a2, symbol Connector_Generic:Conn_01x21
- added J213: b2, symbol Connector_Generic:Conn_01x21
- added J214: c2, symbol Connector_Generic:Conn_01x21
- added J215: d2, symbol Connector_Generic:Conn_01x21
- added J216: e2, symbol Connector_Generic:Conn_01x21
- added J217: f2, symbol Connector_Generic:Conn_01x21
- added J218: g2, symbol Connector_Generic:Conn_01x21
- added J219: a3, symbol Connector_Generic:Conn_01x21
- added J220: b3, symbol Connector_Generic:Conn_01x21
- added J221: c3, symbol Connector_Generic:Conn_01x21
- added J222: d3, symbol Connector_Generic:Conn_01x21
- added J223: e3, symbol Connector_Generic:Conn_01x21
- added J224: f3, symbol Connector_Generic:Conn_01x21
- added J225: g3, symbol Connector_Generic:Conn_01x21
- added J226, J227, J228, J229, J230, J231, J232: a4, symbol Connector_Generic:Conn_01x21
- J101: value a -> a1
- J102: value b -> b1
- J103: value c -> c1
- J104: value d -> d1
- J105: value e -> e1
- J106: value f -> f1
- J107: value g -> a2
- J108: value h -> b2
- J109: value i -> c2
- J110: value j -> d2
- J111: value k -> e2
- J112: value l -> f2
- J113: value m -> a3
- J114: value n -> b3
- J115: value o -> c3
- J116: value p -> d3
- J117: value q -> e3
- J118: value r -> f3
- J119: value s -> a4
- J120: value t -> b4
- J121: value u -> c4
- J122: value v -> d4
- J123: value w -> e4
- J124: value x -> f4
Connections:
- net B1: now also J202.1 (Pin_1)
- net B10: now also J202.10 (Pin_10)
- net B11: now also J202.11 (Pin_11)
- net B12: now also J202.12 (Pin_12)
- net B13: now also J202.13 (Pin_13)
- net B14: now also J202.14 (Pin_14)
- net B15: now also J202.15 (Pin_15)
- net B16: now also J202.16 (Pin_16)
- net B17: now also J202.17 (Pin_17)
- net B18: now also J202.18 (Pin_18)
- net B19: now also J202.19 (Pin_19)
- net B2: now also J202.2 (Pin_2)
- net B20: now also J202.20 (Pin_20)
- net B21: now also J202.21 (Pin_21)
- net B22: now also J202.22 (Pin_22)
- net B23: now also J202.23 (Pin_23)
- net B24: now also J202.24 (Pin_24)
- net B25: now also J202.25 (Pin_25)
- net B26: now also J202.26 (Pin_26)
- net B27: now also J202.27 (Pin_27)
- net B28: now also J202.28 (Pin_28)
- net B29: now also J202.29 (Pin_29)
- net B3: now also J202.3 (Pin_3)
- net B30: now also J202.30 (Pin_30)
- net B31: now also J202.31 (Pin_31)
- net B32: now also J202.32 (Pin_32)
- net B33: now also J202.33 (Pin_33)
- net B34: now also J202.34 (Pin_34)
- net B4: now also J202.4 (Pin_4)
- net B5: now also J202.5 (Pin_5)
- net B6: now also J202.6 (Pin_6)
- net B7: now also J202.7 (Pin_7)
- net B8: now also J202.8 (Pin_8)
- net B9: now also J202.9 (Pin_9)
- net C1: now also J203.1 (Pin_1)
- net C10: now also J203.10 (Pin_10)
- net C11: now also J203.11 (Pin_11)
- net C12: now also J203.12 (Pin_12)
- net C13: now also J203.13 (Pin_13)
- net C14: now also J203.14 (Pin_14)
- net C15: now also J203.15 (Pin_15)
- net C16: now also J203.16 (Pin_16)
- net C17: now also J203.17 (Pin_17)
- net C18: now also J203.18 (Pin_18)
- net C19: now also J203.19 (Pin_19)
- net C2: now also J203.2 (Pin_2)
- net C20: now also J203.20 (Pin_20)
- net C21: now also J203.21 (Pin_21)
- net C22: now also J203.22 (Pin_22)
- net C23: now also J203.23 (Pin_23)
- net C24: now also J203.24 (Pin_24)
- net C25: now also J203.25 (Pin_25)
- net C26: now also J203.26 (Pin_26)
- net C27: now also J203.27 (Pin_27)
- net C28: now also J203.28 (Pin_28)
- net C29: now also J203.29 (Pin_29)
- net C3: now also J203.3 (Pin_3)
- net C30: now also J203.30 (Pin_30)
- net C31: now also J203.31 (Pin_31)
- net C32: now also J203.32 (Pin_32)
- net C33: now also J203.33 (Pin_33)
- net C34: now also J203.34 (Pin_34)
- net C4: now also J203.4 (Pin_4)
- net C5: now also J203.5 (Pin_5)
- net C6: now also J203.6 (Pin_6)
- net C7: now also J203.7 (Pin_7)
- net C8: now also J203.8 (Pin_8)
- net C9: now also J203.9 (Pin_9)
- net D1: now also J204.1 (Pin_1)
- net D10: now also J204.10 (Pin_10)
- net D11: now also J204.11 (Pin_11)
- net D12: now also J204.12 (Pin_12)
- net D13: now also J204.13 (Pin_13)
- net D14: now also J204.14 (Pin_14)
- net D15: now also J204.15 (Pin_15)
- net D16: now also J204.16 (Pin_16)
- net D17: now also J204.17 (Pin_17)
- net D18: now also J204.18 (Pin_18)
- net D19: now also J204.19 (Pin_19)
- net D2: now also J204.2 (Pin_2)
- net D20: now also J204.20 (Pin_20)
- net D21: now also J204.21 (Pin_21)
- net D22: now also J204.22 (Pin_22)
- net D23: now also J204.23 (Pin_23)
- net D24: now also J204.24 (Pin_24)
- net D25: now also J204.25 (Pin_25)
- net D26: now also J204.26 (Pin_26)
- net D27: now also J204.27 (Pin_27)
- net D28: now also J204.28 (Pin_28)
- net D29: now also J204.29 (Pin_29)
- net D3: now also J204.3 (Pin_3)
- net D30: now also J204.30 (Pin_30)
- net D31: now also J204.31 (Pin_31)
- net D32: now also J204.32 (Pin_32)
- net D33: now also J204.33 (Pin_33)
- net D34: now also J204.34 (Pin_34)
- net D4: now also J204.4 (Pin_4)
- net D5: now also J204.5 (Pin_5)
- net D6: now also J204.6 (Pin_6)
- net D7: now also J204.7 (Pin_7)
- net D8: now also J204.8 (Pin_8)
- net D9: now also J204.9 (Pin_9)
- removed net A1: J101.1 (Pin_1), J102.1 (Pin_1), J103.1 (Pin_1), J104.1 (Pin_1), J105.1 (Pin_1), J106.1 (Pin_1)
- removed net A10: J101.10 (Pin_10), J102.10 (Pin_10), J103.10 (Pin_10), J104.10 (Pin_10), J105.10 (Pin_10), J106.10 (Pin_10)
- removed net A11: J101.11 (Pin_11), J102.11 (Pin_11), J103.11 (Pin_11), J104.11 (Pin_11), J105.11 (Pin_11), J106.11 (Pin_11)
- removed net A12: J101.12 (Pin_12), J102.12 (Pin_12), J103.12 (Pin_12), J104.12 (Pin_12), J105.12 (Pin_12), J106.12 (Pin_12)
- removed net A13: J101.13 (Pin_13), J102.13 (Pin_13), J103.13 (Pin_13), J104.13 (Pin_13), J105.13 (Pin_13), J106.13 (Pin_13)
- removed net A14: J101.14 (Pin_14), J102.14 (Pin_14), J103.14 (Pin_14), J104.14 (Pin_14), J105.14 (Pin_14), J106.14 (Pin_14)
- removed net A15: J101.15 (Pin_15), J102.15 (Pin_15), J103.15 (Pin_15), J104.15 (Pin_15), J105.15 (Pin_15), J106.15 (Pin_15)
- removed net A16: J101.16 (Pin_16), J102.16 (Pin_16), J103.16 (Pin_16), J104.16 (Pin_16), J105.16 (Pin_16), J106.16 (Pin_16)
- removed net A17: J101.17 (Pin_17), J102.17 (Pin_17), J103.17 (Pin_17), J104.17 (Pin_17), J105.17 (Pin_17), J106.17 (Pin_17)
- removed net A18: J101.18 (Pin_18), J102.18 (Pin_18), J103.18 (Pin_18), J104.18 (Pin_18), J105.18 (Pin_18), J106.18 (Pin_18)
- removed net A19: J101.19 (Pin_19), J102.19 (Pin_19), J103.19 (Pin_19), J104.19 (Pin_19), J105.19 (Pin_19), J106.19 (Pin_19)
- removed net A2: J101.2 (Pin_2), J102.2 (Pin_2), J103.2 (Pin_2), J104.2 (Pin_2), J105.2 (Pin_2), J106.2 (Pin_2)
- removed net A20: J101.20 (Pin_20), J102.20 (Pin_20), J103.20 (Pin_20), J104.20 (Pin_20), J105.20 (Pin_20), J106.20 (Pin_20)
- removed net A21: J101.21 (Pin_21), J102.21 (Pin_21), J103.21 (Pin_21), J104.21 (Pin_21), J105.21 (Pin_21), J106.21 (Pin_21)
- removed net A22: J101.22 (Pin_22), J102.22 (Pin_22), J103.22 (Pin_22), J104.22 (Pin_22), J105.22 (Pin_22), J106.22 (Pin_22)
- removed net A23: J101.23 (Pin_23), J102.23 (Pin_23), J103.23 (Pin_23), J104.23 (Pin_23), J105.23 (Pin_23), J106.23 (Pin_23)
- removed net A24: J101.24 (Pin_24), J102.24 (Pin_24), J103.24 (Pin_24), J104.24 (Pin_24), J105.24 (Pin_24), J106.24 (Pin_24)
- removed net A25: J101.25 (Pin_25), J102.25 (Pin_25), J103.25 (Pin_25), J104.25 (Pin_25), J105.25 (Pin_25), J106.25 (Pin_25)
- removed net A26: J101.26 (Pin_26), J102.26 (Pin_26), J103.26 (Pin_26), J104.26 (Pin_26), J105.26 (Pin_26), J106.26 (Pin_26)
- removed net A27: J101.27 (Pin_27), J102.27 (Pin_27), J103.27 (Pin_27), J104.27 (Pin_27), J105.27 (Pin_27), J106.27 (Pin_27)
- removed net A28: J101.28 (Pin_28), J102.28 (Pin_28), J103.28 (Pin_28), J104.28 (Pin_28), J105.28 (Pin_28), J106.28 (Pin_28)
- removed net A29: J101.29 (Pin_29), J102.29 (Pin_29), J103.29 (Pin_29), J104.29 (Pin_29), J105.29 (Pin_29), J106.29 (Pin_29)
- removed net A3: J101.3 (Pin_3), J102.3 (Pin_3), J103.3 (Pin_3), J104.3 (Pin_3), J105.3 (Pin_3), J106.3 (Pin_3)
- removed net A30: J101.30 (Pin_30), J102.30 (Pin_30), J103.30 (Pin_30), J104.30 (Pin_30), J105.30 (Pin_30), J106.30 (Pin_30)
- removed net A31: J101.31 (Pin_31), J102.31 (Pin_31), J103.31 (Pin_31), J104.31 (Pin_31), J105.31 (Pin_31), J106.31 (Pin_31)
- removed net A32: J101.32 (Pin_32), J102.32 (Pin_32), J103.32 (Pin_32), J104.32 (Pin_32), J105.32 (Pin_32), J106.32 (Pin_32)
- removed net A33: J101.33 (Pin_33), J102.33 (Pin_33), J103.33 (Pin_33), J104.33 (Pin_33), J105.33 (Pin_33), J106.33 (Pin_33)
- removed net A34: J101.34 (Pin_34), J102.34 (Pin_34), J103.34 (Pin_34), J104.34 (Pin_34), J105.34 (Pin_34), J106.34 (Pin_34)
- removed net A4: J101.4 (Pin_4), J102.4 (Pin_4), J103.4 (Pin_4), J104.4 (Pin_4), J105.4 (Pin_4), J106.4 (Pin_4)
- removed net A5: J101.5 (Pin_5), J102.5 (Pin_5), J103.5 (Pin_5), J104.5 (Pin_5), J105.5 (Pin_5), J106.5 (Pin_5)
- removed net A6: J101.6 (Pin_6), J102.6 (Pin_6), J103.6 (Pin_6), J104.6 (Pin_6), J105.6 (Pin_6), J106.6 (Pin_6)
- removed net A7: J101.7 (Pin_7), J102.7 (Pin_7), J103.7 (Pin_7), J104.7 (Pin_7), J105.7 (Pin_7), J106.7 (Pin_7)
- removed net A8: J101.8 (Pin_8), J102.8 (Pin_8), J103.8 (Pin_8), J104.8 (Pin_8), J105.8 (Pin_8), J106.8 (Pin_8)
- removed net A9: J101.9 (Pin_9), J102.9 (Pin_9), J103.9 (Pin_9), J104.9 (Pin_9), J105.9 (Pin_9), J106.9 (Pin_9)
- new net: J101.1 (Pin_1), J101.10 (Pin_10), J101.11 (Pin_11), J101.12 (Pin_12), J101.13 (Pin_13), J101.14 (Pin_14), J101.15 (Pin_15), J101.16 (Pin_16), J101.17 (Pin_17), J101.18 (Pin_18), J101.19 (Pin_19), J101.2 (Pin_2), J101.20 (Pin_20), J101.21 (Pin_21), J101.22 (Pin_22), J101.23 (Pin_23), J101.24 (Pin_24), J101.25 (Pin_25), J101.26 (Pin_26), J101.27 (Pin_27), J101.28 (Pin_28), J101.29 (Pin_29), J101.3 (Pin_3), J101.30 (Pin_30), J101.31 (Pin_31), J101.32 (Pin_32), J101.33 (Pin_33), J101.34 (Pin_34), J101.4 (Pin_4), J101.5 (Pin_5), J101.6 (Pin_6), J101.7 (Pin_7), J101.8 (Pin_8), J101.9 (Pin_9), J205.1 (Pin_1), J205.10 (Pin_10), J205.11 (Pin_11), J205.12 (Pin_12), J205.13 (Pin_13), J205.14 (Pin_14), J205.15 (Pin_15), J205.16 (Pin_16), J205.17 (Pin_17), J205.18 (Pin_18), J205.19 (Pin_19), J205.2 (Pin_2), J205.20 (Pin_20), J205.21 (Pin_21), J205.3 (Pin_3), J205.4 (Pin_4), J205.5 (Pin_5), J205.6 (Pin_6), J205.7 (Pin_7), J205.8 (Pin_8), J205.9 (Pin_9)
- new net: J102.1 (Pin_1), J102.10 (Pin_10), J102.11 (Pin_11), J102.12 (Pin_12), J102.13 (Pin_13), J102.14 (Pin_14), J102.15 (Pin_15), J102.16 (Pin_16), J102.17 (Pin_17), J102.18 (Pin_18), J102.19 (Pin_19), J102.2 (Pin_2), J102.20 (Pin_20), J102.21 (Pin_21), J102.22 (Pin_22), J102.23 (Pin_23), J102.24 (Pin_24), J102.25 (Pin_25), J102.26 (Pin_26), J102.27 (Pin_27), J102.28 (Pin_28), J102.29 (Pin_29), J102.3 (Pin_3), J102.30 (Pin_30), J102.31 (Pin_31), J102.32 (Pin_32), J102.33 (Pin_33), J102.34 (Pin_34), J102.4 (Pin_4), J102.5 (Pin_5), J102.6 (Pin_6), J102.7 (Pin_7), J102.8 (Pin_8), J102.9 (Pin_9), J206.1 (Pin_1), J206.10 (Pin_10), J206.11 (Pin_11), J206.12 (Pin_12), J206.13 (Pin_13), J206.14 (Pin_14), J206.15 (Pin_15), J206.16 (Pin_16), J206.17 (Pin_17), J206.18 (Pin_18), J206.19 (Pin_19), J206.2 (Pin_2), J206.20 (Pin_20), J206.21 (Pin_21), J206.3 (Pin_3), J206.4 (Pin_4), J206.5 (Pin_5), J206.6 (Pin_6), J206.7 (Pin_7), J206.8 (Pin_8), J206.9 (Pin_9)
- new net: J103.1 (Pin_1), J103.10 (Pin_10), J103.11 (Pin_11), J103.12 (Pin_12), J103.13 (Pin_13), J103.14 (Pin_14), J103.15 (Pin_15), J103.16 (Pin_16), J103.17 (Pin_17), J103.18 (Pin_18), J103.19 (Pin_19), J103.2 (Pin_2), J103.20 (Pin_20), J103.21 (Pin_21), J103.22 (Pin_22), J103.23 (Pin_23), J103.24 (Pin_24), J103.25 (Pin_25), J103.26 (Pin_26), J103.27 (Pin_27), J103.28 (Pin_28), J103.29 (Pin_29), J103.3 (Pin_3), J103.30 (Pin_30), J103.31 (Pin_31), J103.32 (Pin_32), J103.33 (Pin_33), J103.34 (Pin_34), J103.4 (Pin_4), J103.5 (Pin_5), J103.6 (Pin_6), J103.7 (Pin_7), J103.8 (Pin_8), J103.9 (Pin_9), J207.1 (Pin_1), J207.10 (Pin_10), J207.11 (Pin_11), J207.12 (Pin_12), J207.13 (Pin_13), J207.14 (Pin_14), J207.15 (Pin_15), J207.16 (Pin_16), J207.17 (Pin_17), J207.18 (Pin_18), J207.19 (Pin_19), J207.2 (Pin_2), J207.20 (Pin_20), J207.21 (Pin_21), J207.3 (Pin_3), J207.4 (Pin_4), J207.5 (Pin_5), J207.6 (Pin_6), J207.7 (Pin_7), J207.8 (Pin_8), J207.9 (Pin_9)
- new net: J104.1 (Pin_1), J104.10 (Pin_10), J104.11 (Pin_11), J104.12 (Pin_12), J104.13 (Pin_13), J104.14 (Pin_14), J104.15 (Pin_15), J104.16 (Pin_16), J104.17 (Pin_17), J104.18 (Pin_18), J104.19 (Pin_19), J104.2 (Pin_2), J104.20 (Pin_20), J104.21 (Pin_21), J104.22 (Pin_22), J104.23 (Pin_23), J104.24 (Pin_24), J104.25 (Pin_25), J104.26 (Pin_26), J104.27 (Pin_27), J104.28 (Pin_28), J104.29 (Pin_29), J104.3 (Pin_3), J104.30 (Pin_30), J104.31 (Pin_31), J104.32 (Pin_32), J104.33 (Pin_33), J104.34 (Pin_34), J104.4 (Pin_4), J104.5 (Pin_5), J104.6 (Pin_6), J104.7 (Pin_7), J104.8 (Pin_8), J104.9 (Pin_9), J208.1 (Pin_1), J208.10 (Pin_10), J208.11 (Pin_11), J208.12 (Pin_12), J208.13 (Pin_13), J208.14 (Pin_14), J208.15 (Pin_15), J208.16 (Pin_16), J208.17 (Pin_17), J208.18 (Pin_18), J208.19 (Pin_19), J208.2 (Pin_2), J208.20 (Pin_20), J208.21 (Pin_21), J208.3 (Pin_3), J208.4 (Pin_4), J208.5 (Pin_5), J208.6 (Pin_6), J208.7 (Pin_7), J208.8 (Pin_8), J208.9 (Pin_9)
- new net: J105.1 (Pin_1), J105.10 (Pin_10), J105.11 (Pin_11), J105.12 (Pin_12), J105.13 (Pin_13), J105.14 (Pin_14), J105.15 (Pin_15), J105.16 (Pin_16), J105.17 (Pin_17), J105.18 (Pin_18), J105.19 (Pin_19), J105.2 (Pin_2), J105.20 (Pin_20), J105.21 (Pin_21), J105.22 (Pin_22), J105.23 (Pin_23), J105.24 (Pin_24), J105.25 (Pin_25), J105.26 (Pin_26), J105.27 (Pin_27), J105.28 (Pin_28), J105.29 (Pin_29), J105.3 (Pin_3), J105.30 (Pin_30), J105.31 (Pin_31), J105.32 (Pin_32), J105.33 (Pin_33), J105.34 (Pin_34), J105.4 (Pin_4), J105.5 (Pin_5), J105.6 (Pin_6), J105.7 (Pin_7), J105.8 (Pin_8), J105.9 (Pin_9), J209.1 (Pin_1), J209.10 (Pin_10), J209.11 (Pin_11), J209.12 (Pin_12), J209.13 (Pin_13), J209.14 (Pin_14), J209.15 (Pin_15), J209.16 (Pin_16), J209.17 (Pin_17), J209.18 (Pin_18), J209.19 (Pin_19), J209.2 (Pin_2), J209.20 (Pin_20), J209.21 (Pin_21), J209.3 (Pin_3), J209.4 (Pin_4), J209.5 (Pin_5), J209.6 (Pin_6), J209.7 (Pin_7), J209.8 (Pin_8), J209.9 (Pin_9)
- new net: J106.1 (Pin_1), J106.10 (Pin_10), J106.11 (Pin_11), J106.12 (Pin_12), J106.13 (Pin_13), J106.14 (Pin_14), J106.15 (Pin_15), J106.16 (Pin_16), J106.17 (Pin_17), J106.18 (Pin_18), J106.19 (Pin_19), J106.2 (Pin_2), J106.20 (Pin_20), J106.21 (Pin_21), J106.22 (Pin_22), J106.23 (Pin_23), J106.24 (Pin_24), J106.25 (Pin_25), J106.26 (Pin_26), J106.27 (Pin_27), J106.28 (Pin_28), J106.29 (Pin_29), J106.3 (Pin_3), J106.30 (Pin_30), J106.31 (Pin_31), J106.32 (Pin_32), J106.33 (Pin_33), J106.34 (Pin_34), J106.4 (Pin_4), J106.5 (Pin_5), J106.6 (Pin_6), J106.7 (Pin_7), J106.8 (Pin_8), J106.9 (Pin_9), J210.1 (Pin_1), J210.10 (Pin_10), J210.11 (Pin_11), J210.12 (Pin_12), J210.13 (Pin_13), J210.14 (Pin_14), J210.15 (Pin_15), J210.16 (Pin_16), J210.17 (Pin_17), J210.18 (Pin_18), J210.19 (Pin_19), J210.2 (Pin_2), J210.20 (Pin_20), J210.21 (Pin_21), J210.3 (Pin_3), J210.4 (Pin_4), J210.5 (Pin_5), J210.6 (Pin_6), J210.7 (Pin_7), J210.8 (Pin_8), J210.9 (Pin_9)
- new net: J201.1 (Pin_1), J201.10 (Pin_10), J201.11 (Pin_11), J201.12 (Pin_12), J201.13 (Pin_13), J201.14 (Pin_14), J201.15 (Pin_15), J201.16 (Pin_16), J201.17 (Pin_17), J201.18 (Pin_18), J201.19 (Pin_19), J201.2 (Pin_2), J201.20 (Pin_20), J201.21 (Pin_21), J201.22 (Pin_22), J201.23 (Pin_23), J201.24 (Pin_24), J201.25 (Pin_25), J201.26 (Pin_26), J201.27 (Pin_27), J201.28 (Pin_28), J201.29 (Pin_29), J201.3 (Pin_3), J201.30 (Pin_30), J201.31 (Pin_31), J201.32 (Pin_32), J201.33 (Pin_33), J201.34 (Pin_34), J201.4 (Pin_4), J201.5 (Pin_5), J201.6 (Pin_6), J201.7 (Pin_7), J201.8 (Pin_8), J201.9 (Pin_9), J211.1 (Pin_1), J211.10 (Pin_10), J211.11 (Pin_11), J211.12 (Pin_12), J211.13 (Pin_13), J211.14 (Pin_14), J211.15 (Pin_15), J211.16 (Pin_16), J211.17 (Pin_17), J211.18 (Pin_18), J211.19 (Pin_19), J211.2 (Pin_2), J211.20 (Pin_20), J211.21 (Pin_21), J211.3 (Pin_3), J211.4 (Pin_4), J211.5 (Pin_5), J211.6 (Pin_6), J211.7 (Pin_7), J211.8 (Pin_8), J211.9 (Pin_9)
- new net B35: J212.1 (Pin_1), J213.1 (Pin_1), J214.1 (Pin_1), J215.1 (Pin_1), J216.1 (Pin_1), J217.1 (Pin_1), J218.1 (Pin_1)
- new net B36: J212.2 (Pin_2), J213.2 (Pin_2), J214.2 (Pin_2), J215.2 (Pin_2), J216.2 (Pin_2), J217.2 (Pin_2), J218.2 (Pin_2)
- new net B37: J212.3 (Pin_3), J213.3 (Pin_3), J214.3 (Pin_3), J215.3 (Pin_3), J216.3 (Pin_3), J217.3 (Pin_3), J218.3 (Pin_3)
- new net B38: J212.4 (Pin_4), J213.4 (Pin_4), J214.4 (Pin_4), J215.4 (Pin_4), J216.4 (Pin_4), J217.4 (Pin_4), J218.4 (Pin_4)
- new net B39: J212.5 (Pin_5), J213.5 (Pin_5), J214.5 (Pin_5), J215.5 (Pin_5), J216.5 (Pin_5), J217.5 (Pin_5), J218.5 (Pin_5)
- new net B40: J212.6 (Pin_6), J213.6 (Pin_6), J214.6 (Pin_6), J215.6 (Pin_6), J216.6 (Pin_6), J217.6 (Pin_6), J218.6 (Pin_6)
- new net B41: J212.7 (Pin_7), J213.7 (Pin_7), J214.7 (Pin_7), J215.7 (Pin_7), J216.7 (Pin_7), J217.7 (Pin_7), J218.7 (Pin_7)
- new net B42: J212.8 (Pin_8), J213.8 (Pin_8), J214.8 (Pin_8), J215.8 (Pin_8), J216.8 (Pin_8), J217.8 (Pin_8), J218.8 (Pin_8)
- new net B43: J212.9 (Pin_9), J213.9 (Pin_9), J214.9 (Pin_9), J215.9 (Pin_9), J216.9 (Pin_9), J217.9 (Pin_9), J218.9 (Pin_9)
- new net B44: J212.10 (Pin_10), J213.10 (Pin_10), J214.10 (Pin_10), J215.10 (Pin_10), J216.10 (Pin_10), J217.10 (Pin_10), J218.10 (Pin_10)
- new net B45: J212.11 (Pin_11), J213.11 (Pin_11), J214.11 (Pin_11), J215.11 (Pin_11), J216.11 (Pin_11), J217.11 (Pin_11), J218.11 (Pin_11)
- new net B46: J212.12 (Pin_12), J213.12 (Pin_12), J214.12 (Pin_12), J215.12 (Pin_12), J216.12 (Pin_12), J217.12 (Pin_12), J218.12 (Pin_12)
- new net B47: J212.13 (Pin_13), J213.13 (Pin_13), J214.13 (Pin_13), J215.13 (Pin_13), J216.13 (Pin_13), J217.13 (Pin_13), J218.13 (Pin_13)
- new net B48: J212.14 (Pin_14), J213.14 (Pin_14), J214.14 (Pin_14), J215.14 (Pin_14), J216.14 (Pin_14), J217.14 (Pin_14), J218.14 (Pin_14)
- new net B49: J212.15 (Pin_15), J213.15 (Pin_15), J214.15 (Pin_15), J215.15 (Pin_15), J216.15 (Pin_15), J217.15 (Pin_15), J218.15 (Pin_15)
- new net B50: J212.16 (Pin_16), J213.16 (Pin_16), J214.16 (Pin_16), J215.16 (Pin_16), J216.16 (Pin_16), J217.16 (Pin_16), J218.16 (Pin_16)
- new net B51: J212.17 (Pin_17), J213.17 (Pin_17), J214.17 (Pin_17), J215.17 (Pin_17), J216.17 (Pin_17), J217.17 (Pin_17), J218.17 (Pin_17)
- new net B52: J212.18 (Pin_18), J213.18 (Pin_18), J214.18 (Pin_18), J215.18 (Pin_18), J216.18 (Pin_18), J217.18 (Pin_18), J218.18 (Pin_18)
- new net B53: J212.19 (Pin_19), J213.19 (Pin_19), J214.19 (Pin_19), J215.19 (Pin_19), J216.19 (Pin_19), J217.19 (Pin_19), J218.19 (Pin_19)
- new net B54: J212.20 (Pin_20), J213.20 (Pin_20), J214.20 (Pin_20), J215.20 (Pin_20), J216.20 (Pin_20), J217.20 (Pin_20), J218.20 (Pin_20)
- new net B55: J212.21 (Pin_21), J213.21 (Pin_21), J214.21 (Pin_21), J215.21 (Pin_21), J216.21 (Pin_21), J217.21 (Pin_21), J218.21 (Pin_21)
- new net C35: J219.1 (Pin_1), J220.1 (Pin_1), J221.1 (Pin_1), J222.1 (Pin_1), J223.1 (Pin_1), J224.1 (Pin_1), J225.1 (Pin_1)
- new net C36: J219.2 (Pin_2), J220.2 (Pin_2), J221.2 (Pin_2), J222.2 (Pin_2), J223.2 (Pin_2), J224.2 (Pin_2), J225.2 (Pin_2)
- new net C37: J219.3 (Pin_3), J220.3 (Pin_3), J221.3 (Pin_3), J222.3 (Pin_3), J223.3 (Pin_3), J224.3 (Pin_3), J225.3 (Pin_3)
- new net C38: J219.4 (Pin_4), J220.4 (Pin_4), J221.4 (Pin_4), J222.4 (Pin_4), J223.4 (Pin_4), J224.4 (Pin_4), J225.4 (Pin_4)
- new net C39: J219.5 (Pin_5), J220.5 (Pin_5), J221.5 (Pin_5), J222.5 (Pin_5), J223.5 (Pin_5), J224.5 (Pin_5), J225.5 (Pin_5)
- new net C40: J219.6 (Pin_6), J220.6 (Pin_6), J221.6 (Pin_6), J222.6 (Pin_6), J223.6 (Pin_6), J224.6 (Pin_6), J225.6 (Pin_6)
- new net C41: J219.7 (Pin_7), J220.7 (Pin_7), J221.7 (Pin_7), J222.7 (Pin_7), J223.7 (Pin_7), J224.7 (Pin_7), J225.7 (Pin_7)
- new net C42: J219.8 (Pin_8), J220.8 (Pin_8), J221.8 (Pin_8), J222.8 (Pin_8), J223.8 (Pin_8), J224.8 (Pin_8), J225.8 (Pin_8)
- new net C43: J219.9 (Pin_9), J220.9 (Pin_9), J221.9 (Pin_9), J222.9 (Pin_9), J223.9 (Pin_9), J224.9 (Pin_9), J225.9 (Pin_9)
- new net C44: J219.10 (Pin_10), J220.10 (Pin_10), J221.10 (Pin_10), J222.10 (Pin_10), J223.10 (Pin_10), J224.10 (Pin_10), J225.10 (Pin_10)
- new net C45: J219.11 (Pin_11), J220.11 (Pin_11), J221.11 (Pin_11), J222.11 (Pin_11), J223.11 (Pin_11), J224.11 (Pin_11), J225.11 (Pin_11)
- new net C46: J219.12 (Pin_12), J220.12 (Pin_12), J221.12 (Pin_12), J222.12 (Pin_12), J223.12 (Pin_12), J224.12 (Pin_12), J225.12 (Pin_12)
- new net C47: J219.13 (Pin_13), J220.13 (Pin_13), J221.13 (Pin_13), J222.13 (Pin_13), J223.13 (Pin_13), J224.13 (Pin_13), J225.13 (Pin_13)
- new net C48: J219.14 (Pin_14), J220.14 (Pin_14), J221.14 (Pin_14), J222.14 (Pin_14), J223.14 (Pin_14), J224.14 (Pin_14), J225.14 (Pin_14)
- new net C49: J219.15 (Pin_15), J220.15 (Pin_15), J221.15 (Pin_15), J222.15 (Pin_15), J223.15 (Pin_15), J224.15 (Pin_15), J225.15 (Pin_15)
- new net C50: J219.16 (Pin_16), J220.16 (Pin_16), J221.16 (Pin_16), J222.16 (Pin_16), J223.16 (Pin_16), J224.16 (Pin_16), J225.16 (Pin_16)
- new net C51: J219.17 (Pin_17), J220.17 (Pin_17), J221.17 (Pin_17), J222.17 (Pin_17), J223.17 (Pin_17), J224.17 (Pin_17), J225.17 (Pin_17)
- new net C52: J219.18 (Pin_18), J220.18 (Pin_18), J221.18 (Pin_18), J222.18 (Pin_18), J223.18 (Pin_18), J224.18 (Pin_18), J225.18 (Pin_18)
- new net C53: J219.19 (Pin_19), J220.19 (Pin_19), J221.19 (Pin_19), J222.19 (Pin_19), J223.19 (Pin_19), J224.19 (Pin_19), J225.19 (Pin_19)
- new net C54: J219.20 (Pin_20), J220.20 (Pin_20), J221.20 (Pin_20), J222.20 (Pin_20), J223.20 (Pin_20), J224.20 (Pin_20), J225.20 (Pin_20)
- new net C55: J219.21 (Pin_21), J220.21 (Pin_21), J221.21 (Pin_21), J222.21 (Pin_21), J223.21 (Pin_21), J224.21 (Pin_21), J225.21 (Pin_21)
- new net D35: J226.1 (Pin_1), J227.1 (Pin_1), J228.1 (Pin_1), J229.1 (Pin_1), J230.1 (Pin_1), J231.1 (Pin_1), J232.1 (Pin_1)
- new net D36: J226.2 (Pin_2), J227.2 (Pin_2), J228.2 (Pin_2), J229.2 (Pin_2), J230.2 (Pin_2), J231.2 (Pin_2), J232.2 (Pin_2)
- new net D37: J226.3 (Pin_3), J227.3 (Pin_3), J228.3 (Pin_3), J229.3 (Pin_3), J230.3 (Pin_3), J231.3 (Pin_3), J232.3 (Pin_3)
- new net D38: J226.4 (Pin_4), J227.4 (Pin_4), J228.4 (Pin_4), J229.4 (Pin_4), J230.4 (Pin_4), J231.4 (Pin_4), J232.4 (Pin_4)
- new net D39: J226.5 (Pin_5), J227.5 (Pin_5), J228.5 (Pin_5), J229.5 (Pin_5), J230.5 (Pin_5), J231.5 (Pin_5), J232.5 (Pin_5)
- new net D40: J226.6 (Pin_6), J227.6 (Pin_6), J228.6 (Pin_6), J229.6 (Pin_6), J230.6 (Pin_6), J231.6 (Pin_6), J232.6 (Pin_6)
- new net D41: J226.7 (Pin_7), J227.7 (Pin_7), J228.7 (Pin_7), J229.7 (Pin_7), J230.7 (Pin_7), J231.7 (Pin_7), J232.7 (Pin_7)
- new net D42: J226.8 (Pin_8), J227.8 (Pin_8), J228.8 (Pin_8), J229.8 (Pin_8), J230.8 (Pin_8), J231.8 (Pin_8), J232.8 (Pin_8)
- new net D43: J226.9 (Pin_9), J227.9 (Pin_9), J228.9 (Pin_9), J229.9 (Pin_9), J230.9 (Pin_9), J231.9 (Pin_9), J232.9 (Pin_9)
- new net D44: J226.10 (Pin_10), J227.10 (Pin_10), J228.10 (Pin_10), J229.10 (Pin_10), J230.10 (Pin_10), J231.10 (Pin_10), J232.10 (Pin_10)
- new net D45: J226.11 (Pin_11), J227.11 (Pin_11), J228.11 (Pin_11), J229.11 (Pin_11), J230.11 (Pin_11), J231.11 (Pin_11), J232.11 (Pin_11)
- new net D46: J226.12 (Pin_12), J227.12 (Pin_12), J228.12 (Pin_12), J229.12 (Pin_12), J230.12 (Pin_12), J231.12 (Pin_12), J232.12 (Pin_12)
- new net D47: J226.13 (Pin_13), J227.13 (Pin_13), J228.13 (Pin_13), J229.13 (Pin_13), J230.13 (Pin_13), J231.13 (Pin_13), J232.13 (Pin_13)
- new net D48: J226.14 (Pin_14), J227.14 (Pin_14), J228.14 (Pin_14), J229.14 (Pin_14), J230.14 (Pin_14), J231.14 (Pin_14), J232.14 (Pin_14)
- new net D49: J226.15 (Pin_15), J227.15 (Pin_15), J228.15 (Pin_15), J229.15 (Pin_15), J230.15 (Pin_15), J231.15 (Pin_15), J232.15 (Pin_15)
- new net D50: J226.16 (Pin_16), J227.16 (Pin_16), J228.16 (Pin_16), J229.16 (Pin_16), J230.16 (Pin_16), J231.16 (Pin_16), J232.16 (Pin_16)
- new net D51: J226.17 (Pin_17), J227.17 (Pin_17), J228.17 (Pin_17), J229.17 (Pin_17), J230.17 (Pin_17), J231.17 (Pin_17), J232.17 (Pin_17)
- new net D52: J226.18 (Pin_18), J227.18 (Pin_18), J228.18 (Pin_18), J229.18 (Pin_18), J230.18 (Pin_18), J231.18 (Pin_18), J232.18 (Pin_18)
- new net D53: J226.19 (Pin_19), J227.19 (Pin_19), J228.19 (Pin_19), J229.19 (Pin_19), J230.19 (Pin_19), J231.19 (Pin_19), J232.19 (Pin_19)
- new net D54: J226.20 (Pin_20), J227.20 (Pin_20), J228.20 (Pin_20), J229.20 (Pin_20), J230.20 (Pin_20), J231.20 (Pin_20), J232.20 (Pin_20)
- new net D55: J226.21 (Pin_21), J227.21 (Pin_21), J228.21 (Pin_21), J229.21 (Pin_21), J230.21 (Pin_21), J231.21 (Pin_21), J232.21 (Pin_21)
Other:
- moved on the sheet: H101, H102, H103, H104, J1, J101, J102, J103, J104, J105, J106, J107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

Commit message: done extending prototype area
Parts:
- added J233: a1, symbol Connector_Generic:Conn_01x25
- added J234: b1, symbol Connector_Generic:Conn_01x25
- added J235: c1, symbol Connector_Generic:Conn_01x25
- added J236: d1, symbol Connector_Generic:Conn_01x25
- added J237: e1, symbol Connector_Generic:Conn_01x25
- added J238: f1, symbol Connector_Generic:Conn_01x25
- added J239: g1, symbol Connector_Generic:Conn_01x25
- added J240: a2, symbol Connector_Generic:Conn_01x25
- added J241: b2, symbol Connector_Generic:Conn_01x25
- added J242: c2, symbol Connector_Generic:Conn_01x25
- added J243: d2, symbol Connector_Generic:Conn_01x25
- added J244: e2, symbol Connector_Generic:Conn_01x25
- added J245: f2, symbol Connector_Generic:Conn_01x25
- added J246: g2, symbol Connector_Generic:Conn_01x25
- added J247: a3, symbol Connector_Generic:Conn_01x25
- added J248: b3, symbol Connector_Generic:Conn_01x25
- added J249: c3, symbol Connector_Generic:Conn_01x25
- added J250: d3, symbol Connector_Generic:Conn_01x25
- added J251: e3, symbol Connector_Generic:Conn_01x25
- added J252: f3, symbol Connector_Generic:Conn_01x25
- added J253: g3, symbol Connector_Generic:Conn_01x25
- added J254: a4, symbol Connector_Generic:Conn_01x25
- added J255: b4, symbol Connector_Generic:Conn_01x25
- added J256: c4, symbol Connector_Generic:Conn_01x25
- added J257: d4, symbol Connector_Generic:Conn_01x25
- added J258: e4, symbol Connector_Generic:Conn_01x25
- added J259: f4, symbol Connector_Generic:Conn_01x25
- added J260: g4, symbol Connector_Generic:Conn_01x25
Connections:
- new net: J237.1 (Pin_1), J237.10 (Pin_10), J237.11 (Pin_11), J237.12 (Pin_12), J237.13 (Pin_13), J237.14 (Pin_14), J237.15 (Pin_15), J237.16 (Pin_16), J237.17 (Pin_17), J237.18 (Pin_18), J237.19 (Pin_19), J237.2 (Pin_2), J237.20 (Pin_20), J237.21 (Pin_21), J237.22 (Pin_22), J237.23 (Pin_23), J237.24 (Pin_24), J237.25 (Pin_25), J237.3 (Pin_3), J237.4 (Pin_4), J237.5 (Pin_5), J237.6 (Pin_6), J237.7 (Pin_7), J237.8 (Pin_8), J237.9 (Pin_9)
- new net: J235.1 (Pin_1), J235.10 (Pin_10), J235.11 (Pin_11), J235.12 (Pin_12), J235.13 (Pin_13), J235.14 (Pin_14), J235.15 (Pin_15), J235.16 (Pin_16), J235.17 (Pin_17), J235.18 (Pin_18), J235.19 (Pin_19), J235.2 (Pin_2), J235.20 (Pin_20), J235.21 (Pin_21), J235.22 (Pin_22), J235.23 (Pin_23), J235.24 (Pin_24), J235.25 (Pin_25), J235.3 (Pin_3), J235.4 (Pin_4), J235.5 (Pin_5), J235.6 (Pin_6), J235.7 (Pin_7), J235.8 (Pin_8), J235.9 (Pin_9)
- new net: J238.1 (Pin_1), J238.10 (Pin_10), J238.11 (Pin_11), J238.12 (Pin_12), J238.13 (Pin_13), J238.14 (Pin_14), J238.15 (Pin_15), J238.16 (Pin_16), J238.17 (Pin_17), J238.18 (Pin_18), J238.19 (Pin_19), J238.2 (Pin_2), J238.20 (Pin_20), J238.21 (Pin_21), J238.22 (Pin_22), J238.23 (Pin_23), J238.24 (Pin_24), J238.25 (Pin_25), J238.3 (Pin_3), J238.4 (Pin_4), J238.5 (Pin_5), J238.6 (Pin_6), J238.7 (Pin_7), J238.8 (Pin_8), J238.9 (Pin_9)
- new net: J236.1 (Pin_1), J236.10 (Pin_10), J236.11 (Pin_11), J236.12 (Pin_12), J236.13 (Pin_13), J236.14 (Pin_14), J236.15 (Pin_15), J236.16 (Pin_16), J236.17 (Pin_17), J236.18 (Pin_18), J236.19 (Pin_19), J236.2 (Pin_2), J236.20 (Pin_20), J236.21 (Pin_21), J236.22 (Pin_22), J236.23 (Pin_23), J236.24 (Pin_24), J236.25 (Pin_25), J236.3 (Pin_3), J236.4 (Pin_4), J236.5 (Pin_5), J236.6 (Pin_6), J236.7 (Pin_7), J236.8 (Pin_8), J236.9 (Pin_9)
- new net: J234.1 (Pin_1), J234.10 (Pin_10), J234.11 (Pin_11), J234.12 (Pin_12), J234.13 (Pin_13), J234.14 (Pin_14), J234.15 (Pin_15), J234.16 (Pin_16), J234.17 (Pin_17), J234.18 (Pin_18), J234.19 (Pin_19), J234.2 (Pin_2), J234.20 (Pin_20), J234.21 (Pin_21), J234.22 (Pin_22), J234.23 (Pin_23), J234.24 (Pin_24), J234.25 (Pin_25), J234.3 (Pin_3), J234.4 (Pin_4), J234.5 (Pin_5), J234.6 (Pin_6), J234.7 (Pin_7), J234.8 (Pin_8), J234.9 (Pin_9)
- new net: J233.1 (Pin_1), J233.10 (Pin_10), J233.11 (Pin_11), J233.12 (Pin_12), J233.13 (Pin_13), J233.14 (Pin_14), J233.15 (Pin_15), J233.16 (Pin_16), J233.17 (Pin_17), J233.18 (Pin_18), J233.19 (Pin_19), J233.2 (Pin_2), J233.20 (Pin_20), J233.21 (Pin_21), J233.22 (Pin_22), J233.23 (Pin_23), J233.24 (Pin_24), J233.25 (Pin_25), J233.3 (Pin_3), J233.4 (Pin_4), J233.5 (Pin_5), J233.6 (Pin_6), J233.7 (Pin_7), J233.8 (Pin_8), J233.9 (Pin_9)
- new net: J239.1 (Pin_1), J239.10 (Pin_10), J239.11 (Pin_11), J239.12 (Pin_12), J239.13 (Pin_13), J239.14 (Pin_14), J239.15 (Pin_15), J239.16 (Pin_16), J239.17 (Pin_17), J239.18 (Pin_18), J239.19 (Pin_19), J239.2 (Pin_2), J239.20 (Pin_20), J239.21 (Pin_21), J239.22 (Pin_22), J239.23 (Pin_23), J239.24 (Pin_24), J239.25 (Pin_25), J239.3 (Pin_3), J239.4 (Pin_4), J239.5 (Pin_5), J239.6 (Pin_6), J239.7 (Pin_7), J239.8 (Pin_8), J239.9 (Pin_9)
- new net B56: J240.1 (Pin_1), J241.1 (Pin_1), J242.1 (Pin_1), J243.1 (Pin_1), J244.1 (Pin_1), J245.1 (Pin_1), J246.1 (Pin_1)
- new net B57: J240.2 (Pin_2), J241.2 (Pin_2), J242.2 (Pin_2), J243.2 (Pin_2), J244.2 (Pin_2), J245.2 (Pin_2), J246.2 (Pin_2)
- new net B58: J240.3 (Pin_3), J241.3 (Pin_3), J242.3 (Pin_3), J243.3 (Pin_3), J244.3 (Pin_3), J245.3 (Pin_3), J246.3 (Pin_3)
- new net B59: J240.4 (Pin_4), J241.4 (Pin_4), J242.4 (Pin_4), J243.4 (Pin_4), J244.4 (Pin_4), J245.4 (Pin_4), J246.4 (Pin_4)
- new net B60: J240.5 (Pin_5), J241.5 (Pin_5), J242.5 (Pin_5), J243.5 (Pin_5), J244.5 (Pin_5), J245.5 (Pin_5), J246.5 (Pin_5)
- new net B61: J240.6 (Pin_6), J241.6 (Pin_6), J242.6 (Pin_6), J243.6 (Pin_6), J244.6 (Pin_6), J245.6 (Pin_6), J246.6 (Pin_6)
- new net B62: J240.7 (Pin_7), J241.7 (Pin_7), J242.7 (Pin_7), J243.7 (Pin_7), J244.7 (Pin_7), J245.7 (Pin_7), J246.7 (Pin_7)
- new net B63: J240.8 (Pin_8), J241.8 (Pin_8), J242.8 (Pin_8), J243.8 (Pin_8), J244.8 (Pin_8), J245.8 (Pin_8), J246.8 (Pin_8)
- new net B64: J240.9 (Pin_9), J241.9 (Pin_9), J242.9 (Pin_9), J243.9 (Pin_9), J244.9 (Pin_9), J245.9 (Pin_9), J246.9 (Pin_9)
- new net B65: J240.10 (Pin_10), J241.10 (Pin_10), J242.10 (Pin_10), J243.10 (Pin_10), J244.10 (Pin_10), J245.10 (Pin_10), J246.10 (Pin_10)
- new net B66: J240.11 (Pin_11), J241.11 (Pin_11), J242.11 (Pin_11), J243.11 (Pin_11), J244.11 (Pin_11), J245.11 (Pin_11), J246.11 (Pin_11)
- new net B67: J240.12 (Pin_12), J241.12 (Pin_12), J242.12 (Pin_12), J243.12 (Pin_12), J244.12 (Pin_12), J245.12 (Pin_12), J246.12 (Pin_12)
- new net B68: J240.13 (Pin_13), J241.13 (Pin_13), J242.13 (Pin_13), J243.13 (Pin_13), J244.13 (Pin_13), J245.13 (Pin_13), J246.13 (Pin_13)
- new net B69: J240.14 (Pin_14), J241.14 (Pin_14), J242.14 (Pin_14), J243.14 (Pin_14), J244.14 (Pin_14), J245.14 (Pin_14), J246.14 (Pin_14)
- new net B70: J240.15 (Pin_15), J241.15 (Pin_15), J242.15 (Pin_15), J243.15 (Pin_15), J244.15 (Pin_15), J245.15 (Pin_15), J246.15 (Pin_15)
- new net B71: J240.16 (Pin_16), J241.16 (Pin_16), J242.16 (Pin_16), J243.16 (Pin_16), J244.16 (Pin_16), J245.16 (Pin_16), J246.16 (Pin_16)
- new net B72: J240.17 (Pin_17), J241.17 (Pin_17), J242.17 (Pin_17), J243.17 (Pin_17), J244.17 (Pin_17), J245.17 (Pin_17), J246.17 (Pin_17)
- new net B73: J240.18 (Pin_18), J241.18 (Pin_18), J242.18 (Pin_18), J243.18 (Pin_18), J244.18 (Pin_18), J245.18 (Pin_18), J246.18 (Pin_18)
- new net B74: J240.19 (Pin_19), J241.19 (Pin_19), J242.19 (Pin_19), J243.19 (Pin_19), J244.19 (Pin_19), J245.19 (Pin_19), J246.19 (Pin_19)
- new net B75: J240.20 (Pin_20), J241.20 (Pin_20), J242.20 (Pin_20), J243.20 (Pin_20), J244.20 (Pin_20), J245.20 (Pin_20), J246.20 (Pin_20)
- new net B76: J240.21 (Pin_21), J241.21 (Pin_21), J242.21 (Pin_21), J243.21 (Pin_21), J244.21 (Pin_21), J245.21 (Pin_21), J246.21 (Pin_21)
- new net B77: J240.22 (Pin_22), J241.22 (Pin_22), J242.22 (Pin_22), J243.22 (Pin_22), J244.22 (Pin_22), J245.22 (Pin_22), J246.22 (Pin_22)
- new net B78: J240.23 (Pin_23), J241.23 (Pin_23), J242.23 (Pin_23), J243.23 (Pin_23), J244.23 (Pin_23), J245.23 (Pin_23), J246.23 (Pin_23)
- new net B79: J240.24 (Pin_24), J241.24 (Pin_24), J242.24 (Pin_24), J243.24 (Pin_24), J244.24 (Pin_24), J245.24 (Pin_24), J246.24 (Pin_24)
- new net B80: J240.25 (Pin_25), J241.25 (Pin_25), J242.25 (Pin_25), J243.25 (Pin_25), J244.25 (Pin_25), J245.25 (Pin_25), J246.25 (Pin_25)
- new net C56: J247.1 (Pin_1), J248.1 (Pin_1), J249.1 (Pin_1), J250.1 (Pin_1), J251.1 (Pin_1), J252.1 (Pin_1), J253.1 (Pin_1)
- new net C57: J247.2 (Pin_2), J248.2 (Pin_2), J249.2 (Pin_2), J250.2 (Pin_2), J251.2 (Pin_2), J252.2 (Pin_2), J253.2 (Pin_2)
- new net C58: J247.3 (Pin_3), J248.3 (Pin_3), J249.3 (Pin_3), J250.3 (Pin_3), J251.3 (Pin_3), J252.3 (Pin_3), J253.3 (Pin_3)
- new net C59: J247.4 (Pin_4), J248.4 (Pin_4), J249.4 (Pin_4), J250.4 (Pin_4), J251.4 (Pin_4), J252.4 (Pin_4), J253.4 (Pin_4)
- new net C60: J247.5 (Pin_5), J248.5 (Pin_5), J249.5 (Pin_5), J250.5 (Pin_5), J251.5 (Pin_5), J252.5 (Pin_5), J253.5 (Pin_5)
- new net C61: J247.6 (Pin_6), J248.6 (Pin_6), J249.6 (Pin_6), J250.6 (Pin_6), J251.6 (Pin_6), J252.6 (Pin_6), J253.6 (Pin_6)
- new net C62: J247.7 (Pin_7), J248.7 (Pin_7), J249.7 (Pin_7), J250.7 (Pin_7), J251.7 (Pin_7), J252.7 (Pin_7), J253.7 (Pin_7)
- new net C63: J247.8 (Pin_8), J248.8 (Pin_8), J249.8 (Pin_8), J250.8 (Pin_8), J251.8 (Pin_8), J252.8 (Pin_8), J253.8 (Pin_8)
- new net C64: J247.9 (Pin_9), J248.9 (Pin_9), J249.9 (Pin_9), J250.9 (Pin_9), J251.9 (Pin_9), J252.9 (Pin_9), J253.9 (Pin_9)
- new net C65: J247.10 (Pin_10), J248.10 (Pin_10), J249.10 (Pin_10), J250.10 (Pin_10), J251.10 (Pin_10), J252.10 (Pin_10), J253.10 (Pin_10)
- new net C66: J247.11 (Pin_11), J248.11 (Pin_11), J249.11 (Pin_11), J250.11 (Pin_11), J251.11 (Pin_11), J252.11 (Pin_11), J253.11 (Pin_11)
- new net C67: J247.12 (Pin_12), J248.12 (Pin_12), J249.12 (Pin_12), J250.12 (Pin_12), J251.12 (Pin_12), J252.12 (Pin_12), J253.12 (Pin_12)
- new net C68: J247.13 (Pin_13), J248.13 (Pin_13), J249.13 (Pin_13), J250.13 (Pin_13), J251.13 (Pin_13), J252.13 (Pin_13), J253.13 (Pin_13)
- new net C69: J247.14 (Pin_14), J248.14 (Pin_14), J249.14 (Pin_14), J250.14 (Pin_14), J251.14 (Pin_14), J252.14 (Pin_14), J253.14 (Pin_14)
- new net C70: J247.15 (Pin_15), J248.15 (Pin_15), J249.15 (Pin_15), J250.15 (Pin_15), J251.15 (Pin_15), J252.15 (Pin_15), J253.15 (Pin_15)
- new net C71: J247.16 (Pin_16), J248.16 (Pin_16), J249.16 (Pin_16), J250.16 (Pin_16), J251.16 (Pin_16), J252.16 (Pin_16), J253.16 (Pin_16)
- new net C72: J247.17 (Pin_17), J248.17 (Pin_17), J249.17 (Pin_17), J250.17 (Pin_17), J251.17 (Pin_17), J252.17 (Pin_17), J253.17 (Pin_17)
- new net C73: J247.18 (Pin_18), J248.18 (Pin_18), J249.18 (Pin_18), J250.18 (Pin_18), J251.18 (Pin_18), J252.18 (Pin_18), J253.18 (Pin_18)
- new net C74: J247.19 (Pin_19), J248.19 (Pin_19), J249.19 (Pin_19), J250.19 (Pin_19), J251.19 (Pin_19), J252.19 (Pin_19), J253.19 (Pin_19)
- new net C75: J247.20 (Pin_20), J248.20 (Pin_20), J249.20 (Pin_20), J250.20 (Pin_20), J251.20 (Pin_20), J252.20 (Pin_20), J253.20 (Pin_20)
- new net C76: J247.21 (Pin_21), J248.21 (Pin_21), J249.21 (Pin_21), J250.21 (Pin_21), J251.21 (Pin_21), J252.21 (Pin_21), J253.21 (Pin_21)
- new net C77: J247.22 (Pin_22), J248.22 (Pin_22), J249.22 (Pin_22), J250.22 (Pin_22), J251.22 (Pin_22), J252.22 (Pin_22), J253.22 (Pin_22)
- new net C78: J247.23 (Pin_23), J248.23 (Pin_23), J249.23 (Pin_23), J250.23 (Pin_23), J251.23 (Pin_23), J252.23 (Pin_23), J253.23 (Pin_23)
- new net C79: J247.24 (Pin_24), J248.24 (Pin_24), J249.24 (Pin_24), J250.24 (Pin_24), J251.24 (Pin_24), J252.24 (Pin_24), J253.24 (Pin_24)
- new net C80: J247.25 (Pin_25), J248.25 (Pin_25), J249.25 (Pin_25), J250.25 (Pin_25), J251.25 (Pin_25), J252.25 (Pin_25), J253.25 (Pin_25)
- new net D56: J254.1 (Pin_1), J255.1 (Pin_1), J256.1 (Pin_1), J257.1 (Pin_1), J258.1 (Pin_1), J259.1 (Pin_1), J260.1 (Pin_1)
- new net D57: J254.2 (Pin_2), J255.2 (Pin_2), J256.2 (Pin_2), J257.2 (Pin_2), J258.2 (Pin_2), J259.2 (Pin_2), J260.2 (Pin_2)
- new net D58: J254.3 (Pin_3), J255.3 (Pin_3), J256.3 (Pin_3), J257.3 (Pin_3), J258.3 (Pin_3), J259.3 (Pin_3), J260.3 (Pin_3)
- new net D59: J254.4 (Pin_4), J255.4 (Pin_4), J256.4 (Pin_4), J257.4 (Pin_4), J258.4 (Pin_4), J259.4 (Pin_4), J260.4 (Pin_4)
- new net D60: J254.5 (Pin_5), J255.5 (Pin_5), J256.5 (Pin_5), J257.5 (Pin_5), J258.5 (Pin_5), J259.5 (Pin_5), J260.5 (Pin_5)
- new net D61: J254.6 (Pin_6), J255.6 (Pin_6), J256.6 (Pin_6), J257.6 (Pin_6), J258.6 (Pin_6), J259.6 (Pin_6), J260.6 (Pin_6)
- new net D62: J254.7 (Pin_7), J255.7 (Pin_7), J256.7 (Pin_7), J257.7 (Pin_7), J258.7 (Pin_7), J259.7 (Pin_7), J260.7 (Pin_7)
- new net D63: J254.8 (Pin_8), J255.8 (Pin_8), J256.8 (Pin_8), J257.8 (Pin_8), J258.8 (Pin_8), J259.8 (Pin_8), J260.8 (Pin_8)
- new net D64: J254.9 (Pin_9), J255.9 (Pin_9), J256.9 (Pin_9), J257.9 (Pin_9), J258.9 (Pin_9), J259.9 (Pin_9), J260.9 (Pin_9)
- new net D65: J254.10 (Pin_10), J255.10 (Pin_10), J256.10 (Pin_10), J257.10 (Pin_10), J258.10 (Pin_10), J259.10 (Pin_10), J260.10 (Pin_10)
- new net D66: J254.11 (Pin_11), J255.11 (Pin_11), J256.11 (Pin_11), J257.11 (Pin_11), J258.11 (Pin_11), J259.11 (Pin_11), J260.11 (Pin_11)
- new net D67: J254.12 (Pin_12), J255.12 (Pin_12), J256.12 (Pin_12), J257.12 (Pin_12), J258.12 (Pin_12), J259.12 (Pin_12), J260.12 (Pin_12)
- new net D68: J254.13 (Pin_13), J255.13 (Pin_13), J256.13 (Pin_13), J257.13 (Pin_13), J258.13 (Pin_13), J259.13 (Pin_13), J260.13 (Pin_13)
- new net D69: J254.14 (Pin_14), J255.14 (Pin_14), J256.14 (Pin_14), J257.14 (Pin_14), J258.14 (Pin_14), J259.14 (Pin_14), J260.14 (Pin_14)
- new net D70: J254.15 (Pin_15), J255.15 (Pin_15), J256.15 (Pin_15), J257.15 (Pin_15), J258.15 (Pin_15), J259.15 (Pin_15), J260.15 (Pin_15)
- new net D71: J254.16 (Pin_16), J255.16 (Pin_16), J256.16 (Pin_16), J257.16 (Pin_16), J258.16 (Pin_16), J259.16 (Pin_16), J260.16 (Pin_16)
- new net D72: J254.17 (Pin_17), J255.17 (Pin_17), J256.17 (Pin_17), J257.17 (Pin_17), J258.17 (Pin_17), J259.17 (Pin_17), J260.17 (Pin_17)
- new net D73: J254.18 (Pin_18), J255.18 (Pin_18), J256.18 (Pin_18), J257.18 (Pin_18), J258.18 (Pin_18), J259.18 (Pin_18), J260.18 (Pin_18)
- new net D74: J254.19 (Pin_19), J255.19 (Pin_19), J256.19 (Pin_19), J257.19 (Pin_19), J258.19 (Pin_19), J259.19 (Pin_19), J260.19 (Pin_19)
- new net D75: J254.20 (Pin_20), J255.20 (Pin_20), J256.20 (Pin_20), J257.20 (Pin_20), J258.20 (Pin_20), J259.20 (Pin_20), J260.20 (Pin_20)
- new net D76: J254.21 (Pin_21), J255.21 (Pin_21), J256.21 (Pin_21), J257.21 (Pin_21), J258.21 (Pin_21), J259.21 (Pin_21), J260.21 (Pin_21)
- new net D77: J254.22 (Pin_22), J255.22 (Pin_22), J256.22 (Pin_22), J257.22 (Pin_22), J258.22 (Pin_22), J259.22 (Pin_22), J260.22 (Pin_22)
- new net D78: J254.23 (Pin_23), J255.23 (Pin_23), J256.23 (Pin_23), J257.23 (Pin_23), J258.23 (Pin_23), J259.23 (Pin_23), J260.23 (Pin_23)
- new net D79: J254.24 (Pin_24), J255.24 (Pin_24), J256.24 (Pin_24), J257.24 (Pin_24), J258.24 (Pin_24), J259.24 (Pin_24), J260.24 (Pin_24)
- new net D80: J254.25 (Pin_25), J255.25 (Pin_25), J256.25 (Pin_25), J257.25 (Pin_25), J258.25 (Pin_25), J259.25 (Pin_25), J260.25 (Pin_25)
